File: Hardware/IIS3DWB_breakout_beta/IIS3DWB_breakout_beta.kicad_pcb (KiCad board)
At the start: 2 copper layers, 9.6 x 27 mm, 9 parts, among them J1 5051100892, U1 IIS3DWB

Commit message: Add hardware license and fix BOM issues
Other:
- board text added: "Copyright Ryan Jacoby, Cal Poly CPE Department, Cal Poly IME Department 2025. This source describes Open Hardware and is licensed under the CERN-OHL-P v2 You may redistribute and modify this documentation and make products using it under the terms of the CERN-OHL-P v2 (https:/cern.ch/cern-ohl). This documentation is distributed WITHOUT ANY EXPRESS OR IMPLIED WARRANTY, INCLUDING OF MERCHANTABILITY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"
Changed lines of the file:
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@@
+		)
+	)
+	(gr_text "Copyright Ryan Jacoby, Cal Poly CPE Department, Cal Poly IME Department 2025.\n\nThis source describes Open Hardware and is licensed under the CERN-OHL-P v2\n\nYou may redistribute and modify this documentation and make products\nusing it under the terms of the CERN-OHL-P v2 (https:/cern.ch/cern-ohl).\nThis documentation is distributed WITHOUT ANY EXPRESS OR IMPLIED\nWARRANTY, INCLUDING OF MERCHANTABILITY, SATISFACTORY QUALITY\nAND FITNESS FOR A PARTICULAR PURPOSE. Please see the CERN-OHL-P v2\nfor applicable conditions"
+		(at 18.55 197.25 0)
+		(layer "F.Fab")
+		(effects
+			(font
+				(size 1.5 1.5)
+				(thickness 0.3)
+				(bold yes)
+			)
+			(justify left bottom)
 		)
 	)
