File: Hardware/hw_alpha/connectors.kicad_sch (KiCad schematic)
At the start: 41 parts, among them J1 SI-52003-F, J13 3V3_BYPASS, J3 5V_BYPASS, J7 USB4105-GF-A, U2 Ag9905-MTB, U5 TPD1E05U06DPYR, U6 TPD1E05U06DPYR, U7 LM66100DCK, U8 LM66100DCK, U9 TLV1117-33

Commit message: Add hardware license and fix BOM issues
Parts:
- C1, C46: DPN 445-180843-1-ND -> 732-8487-1-ND
Changed lines of the file:
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@@
 			)
 		)
-		(property "DPN" "445-180843-1-ND"
+		(property "DPN" "732-8487-1-ND"
 			(at 238.76 102.87 0)
 			(effects
@@
 			)
 		)
-		(property "DPN" "445-180843-1-ND"
+		(property "DPN" "732-8487-1-ND"
 			(at 223.52 54.61 0)
 			(effects
