File: Hardware/hw_alpha/hw_alpha.kicad_pcb (KiCad board)
At the start: 4 copper layers, 100 x 100 mm, 171 parts, among them J1 SI-52003-F, J10 5051100892, J11 S6B-PH-SM4-TB, J12 UART, J13 3V3_BYPASS, J2 693063010911, J3 5V_BYPASS, J4 SWD, J5 S6B-PH-SM4-TB, J6 S6B-PH-SM4-TB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

Commit message: Add hardware license and fix BOM issues
Other:
- board text added: "Copyright Ryan Jacoby, Cal Poly CPE Department, Cal Poly IME Department 2025. This source describes Open Hardware and is licensed under the CERN-OHL-P v2 You may redistribute and modify this documentation and make products using it under the terms of the CERN-OHL-P v2 (https:/cern.ch/cern-ohl). This documentation is distributed WITHOUT ANY EXPRESS OR IMPLIED WARRANTY, INCLUDING OF MERCHANTABILITY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"
Changed lines of the file:
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@@
+		)
+	)
+	(gr_text "Copyright Ryan Jacoby, Cal Poly CPE Department, Cal Poly IME Department 2025.\n\nThis source describes Open Hardware and is licensed under the CERN-OHL-P v2\n\nYou may redistribute and modify this documentation and make products\nusing it under the terms of the CERN-OHL-P v2 (https:/cern.ch/cern-ohl).\nThis documentation is distributed WITHOUT ANY EXPRESS OR IMPLIED\nWARRANTY, INCLUDING OF MERCHANTABILITY, SATISFACTORY QUALITY\nAND FITNESS FOR A PARTICULAR PURPOSE. Please see the CERN-OHL-P v2\nfor applicable conditions"
+		(at 180.55 167.8 0)
+		(layer "F.Fab")
+		(effects
+			(font
+				(size 1 1)
+				(thickness 0.15)
+			)
+			(justify left bottom)
 		)
 	)
